File: sminchio.kicad_pcb (KiCad board)
At the start: 2 copper layers, 9 parts, among them J1 Screw_Terminal_01x06, Q1 SQ4435EY, Q2 SQ4435EY, U1 LTC4412xS6, U2 LTC4412xS6

Commit message: Update sminchio.kicad_pcb
toccato il pcb
Parts:
- moved R1 43.5 mm to (92.5, 83.2)
- moved D1 39.4 mm to (95.5, 83.3), turned to 90 degrees
- moved R2 31.5 mm to (92.2, 70.5)
- moved D2 28.8 mm to (93.2, 68.3), turned to 180 degrees
- moved U2 4.83 mm to (93.0, 74.7)
- moved U1 4.76 mm to (93.2, 87.4)
- moved Q2 3.94 mm to (87.7, 73.7)
- moved Q1 3.75 mm to (87.7, 86.4)
Routing:
- net +12V: track 0.00 -> 42.6 mm, vias 0 -> 2
- net Net-(J1-Pad4): track 0.00 -> 14.3 mm
- net Net-(J1-Pad6): track 0.00 -> 13.3 mm
- net Net-(Q1-Pad4): track 0.00 -> 10.3 mm
- net Net-(Q2-Pad4): track 0.00 -> 10.1 mm
- net Net-(D2-Pad1): track 0.00 -> 5.12 mm
- net Net-(D1-Pad1): track 0.00 -> 2.60 mm
- net Net-(D1-Pad2): track 0.00 -> 2.58 mm
- net Net-(D2-Pad2): track 0.00 -> 2.47 mm
- net GND: track 0.00 -> 1.90 mm
- added copper zone on F.Cu, net GND
